Commit message: refresh

File: quadruped_description/urdf/quadruped copy.urdf (robot description, URDF)
Before this commit: robot quadruped, 10 links, 9 joints
Links:
- added link back_left_foot, mass 0.001; visual box size=0.01 0.01 0.01
- added link back_right_foot, mass 0.001; visual box size=0.01 0.01 0.01
- added link front_left_foot, mass 0.001; visual box size=0.01 0.01 0.01
- added link front_right_foot, mass 0.001; visual box size=0.01 0.01 0.01
Joints:
- added joint back_left_foot: type fixed, parent back_left_d, child back_left_foot, origin xyz=0.41 0 0 rpy=0 0 0
- added joint back_right_foot: type fixed, parent back_right_d, child back_right_foot, origin xyz=0.41 0 0 rpy=0 0 0
- added joint front_left_foot: type fixed, parent front_left_d, child front_left_foot, origin xyz=0.41 0 0 rpy=0 0 0
- added joint front_right_foot: type fixed, parent front_right_d, child front_right_foot, origin xyz=0.41 0 0 rpy=0 0 0
