Commit message: refresh

File: quadruped_description/urdf/quadruped.urdf (robot description, URDF)
Before this commit: robot quadruped, 10 links, 9 joints
Joints:
- joint front_left_joint1: child front_right_u -> front_left_u; origin xyz=0.11 -0.05 0 rpy=0 0 0 -> xyz=0.11 0.05 0 rpy=0 0 0
- joint front_left_joint2: child front_right_d -> front_left_d; origin xyz=0.4 -0.005 0 rpy=0 0 0 -> xyz=0.4 0.005 0 rpy=0 0 0; parent front_right_u -> front_left_u
- joint front_right_joint1: child front_left_u -> front_right_u; origin xyz=0.11 0.05 0 rpy=0 0 0 -> xyz=0.11 -0.05 0 rpy=0 0 0
- joint front_right_joint2: child front_left_d -> front_right_d; origin xyz=0.4 0.005 0 rpy=0 0 0 -> xyz=0.4 -0.005 0 rpy=0 0 0; parent front_left_u -> front_right_u

Commit message: Corregidas masas e inercias del urdf

File: quadruped_description/urdf/quadruped.urdf (robot description, URDF)
Before this commit: robot quadruped, 10 links, 9 joints
Links:
- link back_left_d: mass 1 -> 0.5
- link back_left_u: mass 1 -> 0.814
- link back_right_d: mass 1 -> 0.5
- link back_right_u: mass 1 -> 0.814
- link body: mass 1 -> 8.4
- link front_left_d: mass 1 -> 0.5
- link front_left_u: mass 1 -> 0.814
- link front_right_d: mass 1 -> 0.5
- link front_right_u: mass 1 -> 0.814
